File: i2cMasterNano/i2cMaster.kicad_pcb (KiCad board)
At the start: 2 copper layers, 77.5 x 99.1 mm, 27 parts, among them J1 Conn_01x04_Male, J10 Conn_01x01, J2 Conn_01x04_Male, J3 Conn_01x04_Male, J4 Conn_01x04_Male, J5 Conn_01x04_Male, J6 Conn_01x04_Male, J7 Conn_01x04_Male, J8 Conn_01x04_Male, J9 Conn_01x01, SW1 SW_DIP_x03, U1 LM7805_TO220, U2 Arduino_Nano_R3

Commit message: sent to seedstudio
Parts:
- U2: footprint konektory:Arduino_Nano_Ethernet -> arduinoNanoEthernet2:Arduino_Nano_Ethernet2
- moved TVS2 40.8 mm to (151.1, 71.1), turned to 180 degrees
- moved C2 27.4 mm to (191.8, 113.0), turned to 90 degrees
- moved U1 4.02 mm to (191.8, 125.7)
- moved D2 4.02 mm to (199.4, 154.9)
- moved J9 3.81 mm to (200.7, 158.8)
- moved TVS1 2.84 mm to (194.3, 154.9)
- moved J10 2.54 mm to (195.6, 158.8)
- moved C1 1.80 mm to (193.0, 134.6)
Routing:
- net GND: track 260.4 -> 227.4 mm
- net +5V: track 254.4 -> 241.9 mm
- net Net-(C1-Pad1): track 62.1 -> 67.6 mm
- net Net-(D5-Pad2): track 7.12 -> 8.15 mm
- net Net-(D2-Pad1): track 20.6 -> 19.9 mm
